Commit message: Refactor and reorganize the ROS 2 navigation stack for Vstone 4WDS Rover X40A
- Updated .gitignore to include new log and install directories.
- Removed obsolete CMakeLists.txt and package.xml files.
- Modified vstone_params.yaml to align with the official fwdsrover_xna_bringup package parameters.
- Updated launch files to integrate micro-ROS agent and vstone odometry publisher.
- Enhanced URDF model to include base footprint for compatibility with official packages.
- Deleted submodule fwdsrover_xna_ros2 as it is no longer needed.
- Created backup copies of CMakeLists.txt and package.xml for reference.
- Added changelogs for fwdsrover_xna and fwdsrover_xna_bringup packages.
- Implemented new CMakeLists.txt and package.xml for fwdsrover_xna and fwdsrover_xna_bringup.
- Developed pub_odom.cpp to publish odometry and TF information for the rover.
- Created launch files for mouse teleoperation and robot setup.
- Added RViz configuration files for visualization of the rover model.

File: src/rover_description/urdf/rover_x40a.urdf.xacro (robot description, xacro)
@@ -7,4 +7,11 @@
   <xacro:property name="wheel_radius" value="0.075"/>
   <xacro:property name="lidar_height" value="0.2"/>
+  <!-- Base Footprint (on ground, compatible with official Vstone package) -->
+  <link name="base_footprint"/>
+  <joint name="base_footprint_joint" type="fixed">
+    <parent link="base_footprint"/>
+    <child link="base_link"/>
+    <origin xyz="0 0 0.075" rpy="0 0 0"/>  <!-- Lift base_link by wheel radius -->
+  </joint>
   <!-- Base Link -->
   <link name="base_link">
