Commit message: Update LiDAR joint origin for improved alignment with base link

File: src/rover_description/urdf/rover_x40a_official.urdf.xacro (robot description, xacro)
@@ -27,5 +27,5 @@
     <parent link="base_link"/>
     <child link="lidar_link"/>
-    <origin xyz="0.1 0 0.2" rpy="0 0 0"/>
+    <origin xyz="0.0 0.17 0.26" rpy="0 0 ${radians(90)}"/>
   </joint>
   <!-- Gazebo plugins for simulation -->
